File: Hardware/Kicad files/AUX CONTROLS.kicad_sch (KiCad schematic)
At the start: 47 parts, among them J601 LED 1, J602 LED 3, J603 HEATER, J604 LED 2, J605 LED 4, J606 LL1 OUT, J607 LL3 OUT, J608 LL2 OUT, J609 LL4 OUT, Q601 IRLB8721PBF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

Commit message: Add files via upload
Parts:
- added JP601, JP602, JP603, JP604: PULL DOWN, Jumper:SolderJumper-2_P1.3mm_Open_RoundedPad1.0x1.5mm, symbol Jumper:SolderJumper_2_Open
- added R612, R613, R614, R615: 470R, Resistor_SMD:R_0805_2012Metric, symbol Device:R
Connections:
- net GND: now also R612.2, R613.2, R614.2, R615.2
- net L1_PWM: now also JP601.2 (B)
- net L2_PWM: now also JP602.2 (B)
- net L3_PWM: now also JP603.2 (B)
- net L4_PWM: now also JP604.2 (B)
- new net: JP602.1 (A), R613.1
- new net: JP601.1 (A), R612.1
- new net: JP603.1 (A), R614.1
- new net: JP604.1 (A), R615.1
