File: Hardware/Kicad files/Control board.kicad_pcb (KiCad board)
At the start: 2 copper layers, 200 x 150 mm, 94 parts, among them J301 M80-5402642, J302 Conn_02x25_Top_Bottom, J401 FLOW SENSOR 1, J402 LIGHT BARRIER 1, J403 FLOW SENSOR 1, J404 LIGHT BARRIER 2, J405 LIGHT BARRIER 3, J406 THERMOCOUPLE 1, J407 LIGHT BARRIER 4, J408 THERMOCOUPLE 2, J501 2604-1104, J502 EXTRUDER 2 M, J503 EXTRUDER 2 M, J504 EXTRUDER 2 M, J505 EXTRUDER 2 M, J601 LED 1, J602 LED 3, J603 HEATER, J604 LED 2, J605 LED 4, J606 LL1 OUT, J607 LL3 OUT, J608 LL2 OUT, J609 LL4 OUT, Q601 IRLB8721PBF, U201 NUCLEO-H753ZI, U301 MAX485_MODULE_5V_LOGIC_TLL_TO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, U501 TMC2209_SILENTSTEPSTICK, U502 TMC2209_SILENTSTEPSTICK, U503 TMC2209_SILENTSTEPSTICK, U504 TMC2209_SILENTSTEPSTICK, U601 MAGIC-LDHM_172946001, U602 MAGIC-LDHM_172946001, U603 MAGIC-LDHM_172946001, U604 MAGIC-LDHM_172946001

Commit message: Add files via upload
Parts:
- removed J302: Conn_02x25_Top_Bottom, Connector_PinSocket_2.54mm:PinSocket_2x25_P2.54mm_Vertical
- removed J408: THERMOCOUPLE 2, Connector_JST:JST_XH_B6B-XH-A_1x06_P2.50mm_Vertical
- added JP601: PULL DOWN, Jumper:SolderJumper-2_P1.3mm_Open_RoundedPad1.0x1.5mm, F.Cu at (85.2, 150.4)
- added JP602: PULL DOWN, Jumper:SolderJumper-2_P1.3mm_Open_RoundedPad1.0x1.5mm, F.Cu at (76.5, 126.2)
- added JP603: PULL DOWN, Jumper:SolderJumper-2_P1.3mm_Open_RoundedPad1.0x1.5mm, F.Cu at (86.0, 74.7)
- added JP604: PULL DOWN, Jumper:SolderJumper-2_P1.3mm_Open_RoundedPad1.0x1.5mm, F.Cu at (77.3, 101.6)
- added R612: 470R, Resistor_SMD:R_0805_2012Metric, F.Cu at (89.5, 150.4)
- added R613: 470R, Resistor_SMD:R_0805_2012Metric, F.Cu at (81.0, 126.2)
- added R614: 470R, Resistor_SMD:R_0805_2012Metric, F.Cu at (90.4, 74.7)
- added R615: 470R, Resistor_SMD:R_0805_2012Metric, F.Cu at (81.4, 101.6)
- J403: value FLOW SENSOR 1 -> FLOW SENSOR 2
- J502: value EXTRUDER 2 M -> EXTRUDER 1 M
- J504: value EXTRUDER 2 M -> FEED 1 M
- J505: value EXTRUDER 2 M -> FEED 2 M
- moved J407 73.3 mm to (107.3, 145.1)
- moved R408 73.2 mm to (116.5, 143.7)
- moved J608 58.6 mm to (114.1, 66.9)
- moved J606 58.1 mm to (113.9, 76.2)
- moved J607 44.1 mm to (114.1, 57.7)
- moved J609 41.8 mm to (114.1, 49.1)
- moved TP401 17.5 mm to (137.2, 100.8)
- moved D401 17.4 mm to (134.1, 99.9)
- moved TP402 17.2 mm to (137.3, 84.3)
- moved D402 17.1 mm to (133.9, 83.4)
- moved J405 9.29 mm to (107.8, 127.3)
- moved R407 9.09 mm to (116.4, 126.1)
- moved R608 8.99 mm to (131.7, 67.8)
- moved R606 8.99 mm to (131.7, 75.8)
- moved R607 8.99 mm to (131.7, 71.8)
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Connections:
- U201 pad CN10_10: PWM1 -> unconnected-(U201F-D3/TIMER_A_PWM3-PadCN10_10)
- U201 pad CN10_11: TEMP 1 OUT -> unconnected-(U201F-A8/ADC_C_IN-PadCN10_11)
- U201 pad CN10_12: M4_EN -> M3_EN
- U201 pad CN10_13: QSPI_CS -> unconnected-(U201F-D26/QSPI_CS-PadCN10_13)
- U201 pad CN10_14: USART_TX -> unconnected-(U201F-D1/USART_A_TX-PadCN10_14)
- U201 pad CN10_15: QSPI_CLK -> unconnected-(U201F-D27/QSPI_CLK-PadCN10_15)
- U201 pad CN10_16: USART_RX -> unconnected-(U201F-D0/USART_A_RX-PadCN10_16)
- U201 pad CN10_18: PWM5 -> unconnected-(U201F-D42/TIMER_A_PWM1N-PadCN10_18)
- U201 pad CN10_19: QSPI_BK3 -> L2_PWM
- U201 pad CN10_2: M4_DIR -> unconnected-(U201F-D7/IO-PadCN10_2)
- U201 pad CN10_20: PWM4 -> unconnected-(U201F-D41/TIMER_A_ETR-PadCN10_20)
- U201 pad CN10_21: QSPI_BK1 -> unconnected-(U201F-D29/QSPI_BK1_IO1-PadCN10_21)
- U201 pad CN10_23: QSPI_BK0 -> unconnected-(U201F-D30/QSPI_BK1_IO0-PadCN10_23)
- U201 pad CN10_24: PWM3 -> unconnected-(U201F-D40/TIMER_A_PWM2N-PadCN10_24)
- U201 pad CN10_25: QSPI_BK2 -> unconnected-(U201F-D31/QSPI_BK1_IO2-PadCN10_25)
- U201 pad CN10_26: M1_PWM -> unconnected-(U201F-D39/TIMER_A_PWM3N-PadCN10_26)
- U201 pad CN10_28: PWM2 -> M3_PWM
- U201 pad CN10_29: PWM7 -> M4_PWM
- U201 pad CN10_30: L4_PWM -> unconnected-(U201F-D37/TIMER_A_BKIN1-PadCN10_30)
- U201 pad CN10_31: HEATER IN -> unconnected-(U201F-D33/TIMER_D_PWM1-PadCN10_31)
- U201 pad CN10_32: M2_PWM -> L1_PWM
- U201 pad CN10_33: PWM6 -> PWM2
- U201 pad CN10_34: PWM8 -> PWM1
- U201 pad CN10_4: L3_PWM -> unconnected-(U201F-D6/TIMER_A_PWM1-PadCN10_4)
- U201 pad CN10_6: M4_PWM -> unconnected-(U201F-D5/TIMER_A_PWM2-PadCN10_6)
- U201 pad CN10_7: F1_OUT -> unconnected-(U201F-A6/ADC_A_IN-PadCN10_7)
- U201 pad CN10_9: F2_OUT -> unconnected-(U201F-A7/ADC_B_IN-PadCN10_9)
- U201 pad CN7_1: M3_EN -> M1_EN
- U201 pad CN7_11: TH_CS2 -> M2_PWM
- U201 pad CN7_14: M3_PWM -> unconnected-(U201E-D11/SPI_A_MOSI/TIM_E_PWM1-PadCN7_14)
- U201 pad CN7_15: TH_CLK2 -> M1_PWM
- U201 pad CN7_16: L2_PWM -> HEATER IN
- U201 pad CN7_18: L1_PWM -> unconnected-(U201E-D9/TIMER_B_PWM2-PadCN7_18)
- U201 pad CN7_19: TH_DO/MISO2 -> unconnected-(U201E-D25/SPI_B_MISO-PadCN7_19)
- U201 pad CN7_2: M2_DIR -> M1_DIR
- U201 pad CN7_20: D5 -> unconnected-(U201E-D8/IO-PadCN7_20)
- U201 pad CN7_3: M3_DIR -> M2_DIR
- U201 pad CN7_5: M1_DIR -> TH_CS1
- U201 pad CN7_7: M1_EN -> unconnected-(U201E-D19/I2S_A_WS-PadCN7_7)
- U201 pad CN7_9: TH_CS1 -> unconnected-(U201E-D20/I2S_B_WS-PadCN7_9)
- U201 pad CN8_14: D2 -> D2 IN
- U201 pad CN8_16: D1 -> D1 IN
- U201 pad CN8_2: unconnected-(U201C-D43/SDMMC_D0-PadCN8_2) -> L3_PWM
- U201 pad CN9_1: A0 -> F2_OUT
- U201 pad CN9_10: unconnected-(U201D-D55/USART_B_CTS-PadCN9_10) -> LB2_OUT
- U201 pad CN9_11: TEMP 2 OUT -> unconnected-(U201D-A5/ADC3_INP6/I2C1_SCL-PadCN9_11)
- U201 pad CN9_13: D6 -> unconnected-(U201D-D72/COMP1_INP-PadCN9_13)
- U201 pad CN9_14: LB1_OUT -> unconnected-(U201D-D56/SAI_A_MCLK-PadCN9_14)
- U201 pad CN9_15: D5 -> unconnected-(U201D-D71/COMP2_INP-PadCN9_15)
- U201 pad CN9_16: LB2_OUT -> unconnected-(U201D-D57/SAI_A_FS-PadCN9_16)
- U201 pad CN9_18: LB3_OUT -> unconnected-(U201D-D58/SAI_A_SCK-PadCN9_18)
- U201 pad CN9_20: LB4_OUT -> unconnected-(U201D-D59/SAI_A_SD-PadCN9_20)
- U201 pad CN9_22: D10 -> unconnected-(U201D-D60/SAI_B_SD-PadCN9_22)
- U201 pad CN9_24: D9 -> unconnected-(U201D-D61/SAI_B_SCK-PadCN9_24)
- U201 pad CN9_25: CAN_RX -> LB3_OUT
- U201 pad CN9_26: D7 -> unconnected-(U201D-D62/SAI_B_MCLK-PadCN9_26)
- U201 pad CN9_27: CAN_TX -> LB4_OUT
- U201 pad CN9_28: D8 -> M3_DIR
- U201 pad CN9_29: D4 -> M4_DIR
- U201 pad CN9_3: A1 -> F1_OUT
- U201 pad CN9_30: D3 -> M4_EN
- U201 pad CN9_5: A2 -> TEMP 1 OUT
- U201 pad CN9_7: A3 -> L4_PWM
- U201 pad CN9_8: unconnected-(U201D-D54/USART_B_RTS-PadCN9_8) -> LB1_OUT
- U201 pad CN9_9: MAX485_CNT -> TEMP 2 OUT
- U503 pad 10: M4_PWM -> M3_PWM
- U503 pad 16: M4_EN -> M3_EN
- U503 pad 9: M4_DIR -> M3_DIR
- U504 pad 10: M3_PWM -> M4_PWM
- U504 pad 16: M3_EN -> M4_EN
- U504 pad 9: M3_DIR -> M4_DIR
Routing:
- net 5V: track 399.8 -> 563.3 mm, vias 1 -> 3
- net L2_PWM: track 0.00 -> 155.3 mm
- net L1_PWM: track 0.00 -> 155.2 mm
- net TX: track 0.00 -> 139.9 mm, vias 0 -> 1
- net RX: track 0.00 -> 126.6 mm, vias 0 -> 1
- net L4_PWM: track 0.00 -> 108.4 mm
- net L3_PWM: track 0.00 -> 97.2 mm
- net D1 IN: track 0.00 -> 88.6 mm
- net M3_DIR: track 0.00 -> 82.6 mm
- net LB1_OUT: track 8.14 -> 88.1 mm, vias 0 -> 1
- net M4_EN: track 0.00 -> 75.1 mm
- net LB2_OUT: track 8.54 -> 83.3 mm
- net M4_DIR: track 0.00 -> 71.8 mm
- net D2 IN: track 0.00 -> 68.4 mm
- net HEATER IN: track 6.79 -> 72.4 mm
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Other:
- board text added: "12V"
- board text added: "24V"
- board text added: "5V"
- board text added: "CONTROL BOARD V2"
- board text added: "GND"
- board text added: "LAUNCH LOCKS"
- board text added: "THERMOCOUPLE"
- board text added: "USER LEDS"
- board text removed: "D1"
- board text removed: "D10"
- board text removed: "D2"
- board text removed: "D3"
- board text removed: "D4"
- board text removed: "D5"
- board text removed: "D6"
- board text removed: "D7"
- board text removed: "D8"
- board text removed: "D9"
- board text removed: "PWM1"
- board text removed: "U_RX"
- board text removed: "U_TX"

Commit message: Add files via upload
Parts:
- moved H502 3.54 mm to (248.0, 159.0)
- moved H503 3.54 mm to (58.0, 159.0)
- moved H501 2.12 mm to (249.0, 18.0)
- moved H504 1.80 mm to (57.0, 18.0)
Connections:
- U201 pad CN10_10: unconnected-(U201F-D3/TIMER_A_PWM3-PadCN10_10) -> LB2_OUT
- U201 pad CN10_12: M3_EN -> LB3_OUT
- U201 pad CN10_14: unconnected-(U201F-D1/USART_A_TX-PadCN10_14) -> LB4_OUT
- U201 pad CN10_19: L2_PWM -> unconnected-(U201F-D28/QSPI_BK1_IO3-PadCN10_19)
- U201 pad CN10_2: unconnected-(U201F-D7/IO-PadCN10_2) -> M3_DIR
- U201 pad CN10_28: M3_PWM -> unconnected-(U201F-D38/TIMER_A_BKIN2-PadCN10_28)
- U201 pad CN10_29: M4_PWM -> L3_PWM
- U201 pad CN10_31: unconnected-(U201F-D33/TIMER_D_PWM1-PadCN10_31) -> L4_PWM
- U201 pad CN10_33: PWM2 -> unconnected-(U201F-D34/TIMER_B_ETR-PadCN10_33)
- U201 pad CN10_34: PWM1 -> L2_PWM
- U201 pad CN10_4: unconnected-(U201F-D6/TIMER_A_PWM1-PadCN10_4) -> M4_EN
- U201 pad CN10_6: unconnected-(U201F-D5/TIMER_A_PWM2-PadCN10_6) -> M4_DIR
- U201 pad CN10_8: unconnected-(U201F-D4/IO-PadCN10_8) -> LB1_OUT
- U201 pad CN7_1: M1_EN -> M1_PWM
- U201 pad CN7_11: M2_PWM -> unconnected-(U201E-D21/I2S_B_MCK-PadCN7_11)
- U201 pad CN7_13: unconnected-(U201E-D22/I2S_B_SD/SPI_B_MOSI-PadCN7_13) -> M1_EN
- U201 pad CN7_14: unconnected-(U201E-D11/SPI_A_MOSI/TIM_E_PWM1-PadCN7_14) -> M1_DIR
- U201 pad CN7_15: M1_PWM -> unconnected-(U201E-D23/I2S_B_CK/SPI_B_SCK-PadCN7_15)
- U201 pad CN7_16: HEATER IN -> M2_EN
- U201 pad CN7_18: unconnected-(U201E-D9/TIMER_B_PWM2-PadCN7_18) -> M2_DIR
- U201 pad CN7_2: M1_DIR -> M2_PWM
- U201 pad CN7_20: unconnected-(U201E-D8/IO-PadCN7_20) -> M3_EN
- U201 pad CN7_3: M2_DIR -> M4_PWM
- U201 pad CN7_4: M2_EN -> M3_PWM
- U201 pad CN7_9: unconnected-(U201E-D20/I2S_B_WS-PadCN7_9) -> HEATER IN
- U201 pad CN8_2: L3_PWM -> unconnected-(U201C-D43/SDMMC_D0-PadCN8_2)
- U201 pad CN9_10: LB2_OUT -> unconnected-(U201D-D55/USART_B_CTS-PadCN9_10)
- U201 pad CN9_2: UART_SCLK -> unconnected-(U201D-D51/USART_B_SCLK-PadCN9_2)
- U201 pad CN9_25: LB3_OUT -> unconnected-(U201D-D67/CAN_RX-PadCN9_25)
- U201 pad CN9_27: LB4_OUT -> unconnected-(U201D-D66/CAN_TX-PadCN9_27)
- U201 pad CN9_28: M3_DIR -> unconnected-(U201D-D63/SAI_B_FS-PadCN9_28)
- U201 pad CN9_29: M4_DIR -> unconnected-(U201D-D65/IO-PadCN9_29)
- U201 pad CN9_30: M4_EN -> unconnected-(U201D-D64/IO-PadCN9_30)
- U201 pad CN9_7: L4_PWM -> unconnected-(U201D-A3/ADC12_INP5-PadCN9_7)
- U201 pad CN9_8: LB1_OUT -> unconnected-(U201D-D54/USART_B_RTS-PadCN9_8)
Routing:
- net LB1_OUT: track 88.1 -> 201.5 mm, vias 1 -> 0
- net L3_PWM: track 97.2 -> 177.5 mm
- net LB4_OUT: track 70.8 -> 149.6 mm, vias 0 -> 1
- net LB3_OUT: track 55.0 -> 125.5 mm, vias 0 -> 1
- net M4_PWM: track 29.6 -> 89.7 mm
- net L4_PWM: track 108.4 -> 161.1 mm
- net M3_DIR: track 82.6 -> 38.2 mm
- net LB2_OUT: track 83.3 -> 124.1 mm, vias 0 -> 1
- net M3_PWM: track 18.3 -> 58.2 mm
- net M4_EN: track 75.1 -> 47.2 mm
- net M1_EN: track 29.8 -> 56.8 mm, vias 0 -> 1
- net M1_PWM: track 45.9 -> 22.8 mm
- net M2_DIR: track 33.3 -> 17.8 mm
- net M4_DIR: track 71.8 -> 62.0 mm
- net M1_DIR: track 16.8 -> 26.0 mm, vias 0 -> 1
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
Commit message: includes the modifications made
Parts:
- removed H501, H502, H503, H504: MountingHole, MountingHole:MountingHole_3.2mm_M3
- removed U301: MAX485_MODULE_5V_LOGIC_TLL_TO_RS-485_CONVERTER, footprints:MODULE_MAX485_MODULE_5V_LOGIC_TLL_TO_RS-485_CONVERTER
- added C301: 10Nf, Capacitor_SMD:C_0805_2012Metric, F.Cu at (98.5, 68.7)
- added C302: 0.47Uf, Capacitor_SMD:C_0805_2012Metric, F.Cu at (89.6, 60.0)
- added C303: 33Uf, Capacitor_SMD:C_0805_2012Metric, F.Cu at (94.2, 60.0)
- added D403: RED, LED_SMD:LED_0805_2012Metric, F.Cu at (125.0, 32.4)
- added D404: BLUE, LED_SMD:LED_0805_2012Metric, F.Cu at (120.0, 32.5)
- added D405: GREEN, LED_SMD:LED_0805_2012Metric, F.Cu at (115.6, 32.5)
- added D406: YELLOW, LED_SMD:LED_0805_2012Metric, F.Cu at (111.3, 32.5)
- added H301: MountingHole, MountingHole:MountingHole_3.2mm_M3_DIN965_Pad, F.Cu at (254.0, 23.0)
- added H302: MountingHole, MountingHole:MountingHole_3.2mm_M3_DIN965_Pad, F.Cu at (65.0, 23.0)
- added H303: MountingHole, MountingHole:MountingHole_3.2mm_M3_DIN965_Pad, F.Cu at (65.0, 262.0)
- added H304: MountingHole, MountingHole:MountingHole_3.2mm_M3_DIN965_Pad, F.Cu at (254.0, 262.0)
- added IC301: THVD1330DR, footprints:SOIC127P600X175-8N, F.Cu at (91.5, 71.4)
- added R301: 120R, Resistor_SMD:R_0805_2012Metric, F.Cu at (91.5, 65.6)
- added R409: R, Resistor_SMD:R_0805_2012Metric, F.Cu at (125.0, 27.4)
- added R410: 860R, Resistor_SMD:R_0805_2012Metric, F.Cu at (120.0, 27.7)
- added R411: R, Resistor_SMD:R_0805_2012Metric, F.Cu at (115.6, 27.6)
- added R412: R, Resistor_SMD:R_0805_2012Metric, F.Cu at (111.3, 27.8)
- added VR301: LM3940IMP-3.3_NOPB, footprints:VREG_LM3940IMP-3.3_NOPB, F.Cu at (91.9, 52.4)
- moved J602 254.9 mm to (249.5, 235.8), turned to 90 degrees
- moved C607 235.5 mm to (237.5, 234.3), turned to 90 degrees
- moved C602 232.6 mm to (220.0, 246.8), turned to 180 degrees
- moved C608 228.6 mm to (232.5, 234.3), turned to 90 degrees
- moved C604 224.4 mm to (220.0, 241.8), turned to 180 degrees
- moved R603 221.9 mm to (228.0, 233.8), turned to -90 degrees
- moved J605 221.5 mm to (249.0, 208.8), turned to 90 degrees
- moved U602 208.7 mm to (217.0, 234.3), turned to 180 degrees
- moved R614 204.7 mm to (229.3, 225.1)
- moved JP603 204.7 mm to (224.8, 225.1)
- moved C615 199.8 mm to (237.0, 207.3), turned to 90 degrees
- moved J604 198.1 mm to (248.5, 182.8), turned to 90 degrees
- moved C616 192.2 mm to (232.6, 207.3), turned to 90 degrees
- moved C610 189.6 mm to (219.5, 219.8), turned to 180 degrees
- moved J601 187.8 mm to (248.2, 160.3), turned to 90 degrees
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Connections:
- J301 pad 21: unconnected-(J301-Pad21) -> 5V
- J301 pad 8: unconnected-(J301-Pad8) -> 5V
- J406 pad 1: 12V -> 5V
- U201 pad CN8_14: D2 IN -> D1 IN
- U201 pad CN8_16: D1 IN -> D2 IN
- U201 pad CN9_2: unconnected-(U201D-D51/USART_B_SCLK-PadCN9_2) -> DE
Routing:
- net 5V: track 563.3 -> 766.7 mm, vias 3 -> 0
- net TX: track 139.9 -> 54.9 mm, vias 1 -> 0
- net L1_PWM: track 155.8 -> 74.7 mm
- net RX: track 126.6 -> 51.2 mm, vias 1 -> 0
- net L2_PWM: track 159.8 -> 85.8 mm
- net DE: track 0.00 -> 61.2 mm, vias 0 -> 1
- net +3V3: track 0.00 -> 57.8 mm, vias 0 -> 4
- net M2_EN: track 19.6 -> 74.3 mm
- net M1_PWM: track 22.8 -> 77.5 mm
- net M1_DIR: track 26.0 -> 77.9 mm, vias 1 -> 0
- net M2_DIR: track 17.8 -> 68.0 mm
- net L4_PWM: track 161.1 -> 112.2 mm
- net L3_PWM: track 177.5 -> 132.3 mm
- net M3_EN: track 24.2 -> 64.0 mm
- net LB1_OUT: track 201.5 -> 163.1 mm
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Other:
- board size 200 x 150 mm -> 200 x 250 mm
