File: Hardware/Kicad files/Motor Controls.kicad_sch (KiCad schematic)
At the start: 21 parts, among them J501 2604-1104, J502 EXTRUDER 2 M, J503 EXTRUDER 2 M, J504 EXTRUDER 2 M, J505 EXTRUDER 2 M, U501 TMC2209_SILENTSTEPSTICK, U502 TMC2209_SILENTSTEPSTICK, U503 TMC2209_SILENTSTEPSTICK, U504 TMC2209_SILENTSTEPSTICK

Commit message: Add files via upload
Parts:
- J502: value EXTRUDER 2 M -> EXTRUDER 1 M
- J504: value EXTRUDER 2 M -> FEED 1 M
- J505: value EXTRUDER 2 M -> FEED 2 M
Connections:
- net M3_DIR: now also U503.9 (DIR); no longer U504.9 (DIR)
- net M3_EN: now also U503.16 (~{EN}); no longer U504.16 (~{EN})
- net M3_PWM: now also U503.10 (STEP); no longer U504.10 (STEP)
- net M4_DIR: now also U504.9 (DIR); no longer U503.9 (DIR)
- net M4_EN: now also U504.16 (~{EN}); no longer U503.16 (~{EN})
- net M4_PWM: now also U504.10 (STEP); no longer U503.10 (STEP)
Changed lines of the file:
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@@
 	(global_label "M3_EN"
 		(shape input)
-		(at 207.01 114.3 180)
+		(at 203.2 41.91 180)
 		(fields_autoplaced yes)
 		(effects
@@
 		)
 		(property "Intersheetrefs" "${INTERSHEET_REFS}"
-			(at 197.9168 114.3 0)
+			(at 194.1068 41.91 0)
 			(effects
 				(font
@@
 	(global_label "M4_PWM"
 		(shape input)
-		(at 203.2 46.99 180)
+		(at 207.01 119.38 180)
 		(fields_autoplaced yes)
 		(effects
@@
 		)
 		(property "Intersheetrefs" "${INTERSHEET_REFS}"
-			(at 192.4135 46.99 0)
+			(at 196.2235 119.38 0)
 			(effects
 				(font
@@
 	(global_label "M3_PWM"
 		(shape input)
-		(at 207.01 119.38 180)
+		(at 203.2 46.99 180)
 		(fields_autoplaced yes)
 		(effects
@@
 		)
 		(property "Intersheetrefs" "${INTERSHEET_REFS}"
-			(at 196.2235 119.38 0)
+			(at 192.4135 46.99 0)
 			(effects
 				(font
@@
 	(global_label "M4_DIR"
 		(shape input)
-		(at 203.2 49.53 180)
+		(at 207.01 121.92 180)
 		(fields_autoplaced yes)
 		(effects
@@
 		)
 		(property "Intersheetrefs" "${INTERSHEET_REFS}"
-			(at 194.1068 49.53 0)
+			(at 197.9168 121.92 0)
 			(effects
 				(font
@@
 	(global_label "M3_DIR"
 		(shape input)
-		(at 207.01 121.92 180)
+		(at 203.2 49.53 180)
 		(fields_autoplaced yes)
 		(effects
@@
 		)
 		(property "Intersheetrefs" "${INTERSHEET_REFS}"
-			(at 197.9168 121.92 0)
+			(at 194.1068 49.53 0)
 			(effects
 				(font
@@
 	(global_label "M4_EN"
 		(shape input)
-		(at 203.2 41.91 180)
+		(at 207.01 114.3 180)
 		(fields_autoplaced yes)
 		(effects
@@
 		)
 		(property "Intersheetrefs" "${INTERSHEET_REFS}"
-			(at 194.1068 41.91 0)
+			(at 197.9168 114.3 0)
 			(effects
 				(font
@@
 			)
 		)
-		(property "Value" "EXTRUDER 2 M"
+		(property "Value" "EXTRUDER 1 M"
 			(at 156.21 46.99 0)
 			(effects
@@
 			)
 		)
-		(property "Value" "EXTRUDER 2 M"
+		(property "Value" "FEED 2 M"
 			(at 255.27 119.38 0)
 			(effects
@@
 			)
 		)
-		(property "Value" "EXTRUDER 2 M"
+		(property "Value" "FEED 1 M"
 			(at 251.46 46.99 0)
 			(effects

Commit message: includes the modifications made
Parts:
- removed H501, H502, H503, H504: MountingHole, MountingHole:MountingHole_3.2mm_M3, symbol Mechanical:MountingHole
Other:
- note removed: "MOUNTING HOLES"
