File: Hardware/Kicad files/Sensors.kicad_sch (KiCad schematic)
At the start: 20 parts, among them J401 FLOW SENSOR 1, J402 LIGHT BARRIER 1, J403 FLOW SENSOR 1, J404 LIGHT BARRIER 2, J405 LIGHT BARRIER 3, J406 THERMOCOUPLE 1, J407 LIGHT BARRIER 4, J408 THERMOCOUPLE 2

Commit message: Add files via upload
Parts:
- removed J408: THERMOCOUPLE 2, Connector_JST:JST_XH_B6B-XH-A_1x06_P2.50mm_Vertical, symbol Connector:Conn_01x06_Pin
- J403: value FLOW SENSOR 1 -> FLOW SENSOR 2
Connections:
- no-connect marks 6 -> 5

Commit message: includes the modifications made
Parts:
- added D403: RED, LED_SMD:LED_0805_2012Metric, symbol Device:LED
- added D404: BLUE, LED_SMD:LED_0805_2012Metric, symbol Device:LED
- added D405: GREEN, LED_SMD:LED_0805_2012Metric, symbol Device:LED
- added D406: YELLOW, LED_SMD:LED_0805_2012Metric, symbol Device:LED
- added R409: 1.2K 1/2W, Resistor_SMD:R_0805_2012Metric, symbol Device:R
- added R410: 620R, Resistor_SMD:R_0805_2012Metric, symbol Device:R
- added R411: 220R, Resistor_SMD:R_0805_2012Metric, symbol Device:R
- added R412: 130R, Resistor_SMD:R_0805_2012Metric, symbol Device:R
Connections:
- net 12V: now also D404.2 (A); no longer J406.1 (Pin_1)
- net 24V: now also D403.2 (A)
- net 5V: now also J406.1 (Pin_1), D405.2 (A)
- net GND: now also R409.2, R410.2, R411.2, R412.2
- new net: D403.1 (K), R409.1
- new net: D404.1 (K), R410.1
- new net: D406.1 (K), R412.1
- new net: D405.1 (K), R411.1
- new net +3V3: D406.2 (A)
Other:
- note added: "STATUS LEDS"
