File: Hardware/Kicad files/comm.kicad_sch (KiCad schematic)
At the start: 5 parts, among them J301 M80-5402642, J302 Conn_02x25_Top_Bottom, U301 MAX485_MODULE_5V_LOGIC_TLL_TO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

Commit message: Add files via upload
Parts:
- removed J302: Conn_02x25_Top_Bottom, Connector_PinSocket_2.54mm:PinSocket_2x25_P2.54mm_Vertical, symbol Connector_Generic:Conn_02x25_Top_Bottom
Connections:
- no-connect marks 29 -> 16
Other:
- note removed: "GENERAL PURPOSE PORTS"

Commit message: includes the modifications made
Parts:
- removed U301: MAX485_MODULE_5V_LOGIC_TLL_TO_RS-485_CONVERTER, footprints:MODULE_MAX485_MODULE_5V_LOGIC_TLL_TO_RS-485_CONVERTER, symbol MAX485_MODULE_5V_LOGIC_TLL_TO_RS-485_CONVERTER:MAX485_MODULE_5V_LOGIC_TLL_TO_RS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
- added C301: 10Nf, Capacitor_SMD:C_0805_2012Metric, symbol Device:C
- added C302: 0.47Uf, Capacitor_SMD:C_0805_2012Metric, symbol Device:C
- added C303: 33Uf, Capacitor_SMD:C_0805_2012Metric, symbol Device:C
- added H301, H302, H303, H304: MountingHole, MountingHole:MountingHole_3.2mm_M3_DIN965_Pad, symbol Mechanical:MountingHole
- added IC301: THVD1330DR, footprints:SOIC127P600X175-8N, symbol THVD1330DR:THVD1330DR
- added R301: 120R, Resistor_SMD:R_0805_2012Metric, symbol Device:R
- added VR301: LM3940IMP-3.3_NOPB, footprints:VREG_LM3940IMP-3.3_NOPB, symbol LM3940IMP-3.3_NOPB:LM3940IMP-3.3_NOPB
Connections:
- net 5V: now also J301.21, J301.8, C302.1, VR301.1 (IN)
- net GND: now also C301.2, C302.2, C303.2, IC301.5 (GND), VR301.2 (GND_2), VR301.4 (GND_4)
- net RS485_A: now also IC301.7 (B), R301.1
- net RS485_B: now also IC301.6 (A), R301.2
- net RX: now also IC301.4 (D)
- net TX: now also IC301.1 (R)
- new net +3V3: C301.1, C303.1, IC301.8 (VCC), VR301.3 (OUT)
- new net DE: IC301.2 (~{RE}), IC301.3 (DE)
- no-connect marks 16 -> 14
Other:
- note added: "3.3V REGULATOR"
- note added: "MOUNTING HOLES"
